Commit message: working version

File: urdf/kamagami.xacro (robot description, xacro)
@@ -10,18 +10,4 @@
 </xacro:macro>
 <xacro:property name="wheel_radius" value="0.03" />
-	<link name="base_footprint_link">
-		<inertial>
-			<mass value="0.001"/>
-			<inertia
-				ixx="0.0001" ixy="0.0" ixz="0.0"
-				iyy="0.0001" iyz="0.0"
-				izz="0.0001"/>
-		</inertial>
-	</link>
-	<joint name="base_footprint_joint" type="fixed">
-		<origin xyz="0 0 ${wheel_radius}"/>
-		<child link="base_link"/>
-		<parent link="base_footprint_link"/>
-	</joint>
 	<link name="base_link">
 		<collision>
@@ -80,7 +66,7 @@
 		</joint>
 	</xacro:macro>
-	<xacro:wheel name="left_wheel" xyz="0.0 -0.03 0"
+	<xacro:wheel name="left_wheel" xyz="0.0 0.03 0"
 		rpy="1.5708 0 0"/>
-	<xacro:wheel name="right_wheel" xyz="0.0 0.03 0"
+	<xacro:wheel name="right_wheel" xyz="0.0 -0.03 0"
 		rpy="1.5708 0 0"/>
 	<link name="raspicam_link">
@@ -145,7 +131,7 @@
 	    <wheelSeparation>0.14</wheelSeparation>
 	    <wheelAcceleration>0</wheelAcceleration>
-	    <wheelTorque>5</wheelTorque>
+	    <wheelTorque>1</wheelTorque>
 	    <wheelDiameter>0.06</wheelDiameter>
-	    <torque>5</torque>
+	    <torque>1</torque>
 	    <commandTopic>cmd_vel</commandTopic>
 	    <odometryTopic>odom</odometryTopic>

File: urdf/materials.xacro (robot description, xacro)
@@ -14,5 +14,5 @@
   </material>
   <material name="orange">
-    <color rgba="${255/255} ${108/255} ${10/255} 1.0"/>
+    <color rgba="${255/255} ${108/255} ${10/255} 0.5"/>
   </material>
   <material name="brown">

Commit message: fixed kamagmi for correct velocities

File: urdf/kamagami.xacro (robot description, xacro)
@@ -1,13 +1,88 @@
 <?xml version="1.0"?>
 <robot xmlns:xacro="http://www.ros.org/wiki/xacro" name="roadrunner">
-<xacro:macro name="ball_wheel" params="origin">
+<xacro:property name="wheel_radius" value="0.03" />
+<xacro:property name="wheel_separation" value="0.12" />
+<xacro:property name="show_wheels" value="false" />
+<xacro:macro name="ball_wheel" params="origin name">
+	<link name="${name}_link">
 		<collision>
-			<origin xyz="${origin}"/>
 			<geometry>
 				<sphere radius="0.005"/>
 			</geometry>
 		</collision>
+			<inertial>
+				<mass value="0.01"/>
+				<inertia
+					ixx="0.000001" ixy="0.0" ixz="0.0"
+					iyy="0.000001" iyz="0.0"
+					izz="0.000001" />
+			</inertial>
+		<xacro:if value="${show_wheels}">
+			<visual>
+				<geometry>
+					<sphere radius="0.005"/>
+				</geometry>
+			</visual>
+		</xacro:if>
+	</link>
+		<gazebo reference="${name}_link">
+			<material>Gazebo/Orange</material>
+			<mu1 value="0.1"/>
+			<mu2 value="0.1"/>
+		</gazebo>
+		<joint name="${name}_joint" type="fixed">
+			<origin xyz="${origin}"/>
+			<parent link="base_link"/>
+			<child link="${name}_link"/>
+		</joint>
 </xacro:macro>
-<xacro:property name="wheel_radius" value="0.03" />
+	<xacro:macro name="wheel" params="xyz rpy name">
+		<link name="${name}_link">
+			<collision name="collision">
+				<geometry>
+					<cylinder radius="${wheel_radius}" length="0.01"/>
+				</geometry>
+			</collision>
+			<inertial>
+				<mass value="0.01"/>
+				<inertia
+					ixx="0.000001" ixy="0.0" ixz="0.0"
+					iyy="0.000001" iyz="0.0"
+					izz="0.000001" />
+			</inertial>
+		<xacro:if value="${show_wheels}">
+			<visual>
+				<geometry>
+					<cylinder radius="${wheel_radius}" length="0.01"/>
+				</geometry>
+			</visual>
+		</xacro:if>
+		</link>
+		<gazebo reference="${name}_link">
+			<material>Gazebo/Orange</material>
+			<mu1 value="0.8"/>
+			<mu2 value="0.8"/>
+		</gazebo>
+		<joint name="${name}_joint" type="continuous">
+			<origin xyz="${xyz}" rpy="${rpy}"/>
+			<parent link="base_link"/>
+			<child link="${name}_link"/>
+			<axis xyz="0 0 -1"/>
+		</joint>
+	</xacro:macro>
+	<link name="base_footprint_link">
+			<inertial>
+				<mass value="0.01"/>
+				<inertia
+					ixx="0.000001" ixy="0.0" ixz="0.0"
+					iyy="0.000001" iyz="0.0"
+					izz="0.000001" />
+			</inertial>
+	</link>
+		<joint name="base_joint" type="fixed">
+			<origin xyz="0 0 0.025"/>
+			<parent link="base_footprint_link"/>
+			<child link="base_link"/>
+		</joint>
 	<link name="base_link">
 		<collision>
@@ -23,5 +98,4 @@
 				</geometry>
 		</visual>
-		<xacro:ball_wheel origin="-0.05 0 -0.024"/>
 		<inertial>
 			<origin xyz="0 0 0"/>
@@ -34,38 +108,10 @@
 	</link>
 	<gazebo reference="base_link">
-			<mu1 value="0.001"/>
-			<mu2 value="0.001"/>
 		<material>Gazebo/Black</material>
 	</gazebo>
-	<xacro:macro name="wheel" params="xyz rpy name">
-		<link name="${name}_link">
-			<collision name="collision">
-				<geometry>
-					<cylinder radius="${wheel_radius}" length="0.067"/>
-				</geometry>
-			</collision>
-			<inertial>
-				<mass value="0.01"/>
-				<inertia
-					ixx="0.000001" ixy="0.0" ixz="0.0"
-					iyy="0.000001" iyz="0.0"
-					izz="0.000001" />
-			</inertial>
-		</link>
-		<gazebo reference="${name}_link">
-			<material>Gazebo/Orange</material>
-			<mu1 value="0.8"/>
-			<mu2 value="0.8"/>
-		</gazebo>
-		<joint name="${name}_joint" type="continuous">
-			<origin xyz="${xyz}" rpy="${rpy}"/>
-			<parent link="base_link"/>*
-			<child link="${name}_link"/>
-			<axis xyz="0 0 -1"/>
-		</joint>
-	</xacro:macro>
-	<xacro:wheel name="left_wheel" xyz="0.05 -0.03 0"
+	<xacro:ball_wheel origin="-0.05 0 -0.025" name="ball"/>
+	<xacro:wheel name="left_wheel" xyz="0.05 ${wheel_separation/2.0} 0"
 		rpy="1.5708 0 0"/>
-	<xacro:wheel name="right_wheel" xyz="0.05 0.03 0"
+	<xacro:wheel name="right_wheel" xyz="0.05 -${wheel_separation/2.0} 0"
 		rpy="1.5708 0 0"/>
 	<link name="raspicam_link">
@@ -128,8 +174,6 @@
 	    <leftJoint>left_wheel_joint</leftJoint>
 	    <rightJoint>right_wheel_joint</rightJoint>
-	    <wheelSeparation>0.14</wheelSeparation>
 	    <wheelAcceleration>0</wheelAcceleration>
 	    <wheelTorque>1</wheelTorque>
-	    <wheelDiameter>0.06</wheelDiameter>
 	    <torque>1</torque>
 	    <commandTopic>cmd_vel</commandTopic>

File: urdf/kamagami_with_cone.xacro (robot description, xacro)
@@ -11,5 +11,5 @@
 </link>
 <gazebo reference="cone_link">
-	<material>Gazebo/YellowTransparent</material>
+	<material value="Gazebo/YellowTransparent"/>
 </gazebo>
 <joint name="cone_joint" type="fixed">

Commit message: renamed frame for base_link

File: urdf/kamagami.xacro (robot description, xacro)
@@ -3,5 +3,5 @@
 <xacro:property name="wheel_radius" value="0.03" />
 <xacro:property name="wheel_separation" value="0.12" />
-<xacro:property name="show_wheels" value="false" />
+<xacro:property name="show_wheels" value="true" />
 <xacro:macro name="ball_wheel" params="origin name">
 	<link name="${name}_link">
@@ -33,5 +33,5 @@
 		<joint name="${name}_joint" type="fixed">
 			<origin xyz="${origin}"/>
-			<parent link="base_link"/>
+			<parent link="body_link"/>
 			<child link="${name}_link"/>
 		</joint>
@@ -66,10 +66,10 @@
 		<joint name="${name}_joint" type="continuous">
 			<origin xyz="${xyz}" rpy="${rpy}"/>
-			<parent link="base_link"/>
+			<parent link="body_link"/>
 			<child link="${name}_link"/>
 			<axis xyz="0 0 -1"/>
 		</joint>
 	</xacro:macro>
-	<link name="base_footprint_link">
+	<link name="base_link">
 			<inertial>
 				<mass value="0.01"/>
@@ -82,8 +82,8 @@
 		<joint name="base_joint" type="fixed">
 			<origin xyz="0 0 0.025"/>
-			<parent link="base_footprint_link"/>
-			<child link="base_link"/>
+			<parent link="base_link"/>
+			<child link="body_link"/>
 		</joint>
-	<link name="base_link">
+	<link name="body_link">
 		<collision>
 			<origin xyz="0 0 0"/>
@@ -107,5 +107,5 @@
 		</inertial>
 	</link>
-	<gazebo reference="base_link">
+	<gazebo reference="body_link">
 		<material>Gazebo/Black</material>
 	</gazebo>
@@ -123,5 +123,5 @@
 	</link>
 	<joint name="raspicam_joint" type="fixed">
-		<parent link="base_link"/>
+		<parent link="body_link"/>
 		<child link="raspicam_link"/>
 		<origin xyz="0.05 0 0.02" rpy="0 0 0"/>
@@ -182,5 +182,5 @@
 	    <odometryFrame>odom</odometryFrame>
 	    <rosDebugLevel>none</rosDebugLevel>
-	    <robotBaseFrame>base_footprint_link</robotBaseFrame>
+	    <robotBaseFrame>base_link</robotBaseFrame>
 			<updateRate>10</updateRate>
 	  </plugin>

Commit message: stop displaying wheels

File: urdf/kamagami.xacro (robot description, xacro)
@@ -3,5 +3,5 @@
 <xacro:property name="wheel_radius" value="0.03" />
 <xacro:property name="wheel_separation" value="0.12" />
-<xacro:property name="show_wheels" value="true" />
+<xacro:property name="show_wheels" value="false" />
 <xacro:macro name="ball_wheel" params="origin name">
 	<link name="${name}_link">

Commit message: added laser

File: urdf/kamagami.xacro (robot description, xacro)
@@ -186,3 +186,55 @@
 	  </plugin>
 	</gazebo>
+  <joint name="laser_joint" type="fixed">
+    <axis xyz="0 1 0" />
+    <origin xyz="0 0 0.03" rpy="0 0 0"/>
+    <parent link="body_link"/>
+    <child link="laser_link"/>
+  </joint>
+  <!-- Hokuyo Laser -->
+  <link name="laser_link">
+    <collision>
+      <origin xyz="0 0 0" rpy="0 0 0"/>
+      <geometry>
+    <box size="0.1 0.1 0.1"/>
+      </geometry>
+    </collision>
+    <inertial>
+      <mass value="1e-5" />
+      <origin xyz="0 0 0" rpy="0 0 0"/>
+      <inertia ixx="1e-6" ixy="0" ixz="0" iyy="1e-6" iyz="0" izz="1e-6" />
+    </inertial>
+  </link>
+    <gazebo reference="laser_link">
+        <sensor name="laser" type="ray">
+        <pose>0 0 0 0 0 0</pose>
+          <ray>
+            <scan>
+              <horizontal>
+                <!-- The URG-04LX-UG01  has  683 steps with 0.35139 Degree resolution -->
+                <resolution>1</resolution>
+                <max_angle>2.0944</max_angle> <!-- 120 Degree -->
+                <min_angle>-2.0944</min_angle> <!-- -120 Degree -->
+                <samples>683</samples>
+              </horizontal>
+            </scan>
+            <range>
+              <min>0.08</min>
+              <max>5</max>
+              <resolution>0.01</resolution>
+            </range>
+          </ray>
+          <plugin name="laser" filename="libgazebo_ros_laser.so" >
+            <robotNamespace></robotNamespace>
+            <topicName>scan</topicName>
+            <frameName>laser_link</frameName>
+          </plugin>
+          <!--
+          <plugin name="laser" filename="libRayPlugin.so" />
+          -->
+          <always_on>1</always_on>
+          <update_rate>30</update_rate>
+          <visualize>true</visualize>
+        </sensor>
+    </gazebo>
 </robot>

Commit message: tweaked diff drive params and raised laser above camera

File: urdf/kamagami.xacro (robot description, xacro)
@@ -170,10 +170,10 @@
 	    <legacyMode>false</legacyMode>
 	    <publishWheelTF>false</publishWheelTF>
-	    <publishTf>0</publishTf>
-	    <publishWheelJointState>true</publishWheelJointState>
+	    <publishTf>false</publishTf>
+	    <publishWheelJointState>false</publishWheelJointState>
 	    <leftJoint>left_wheel_joint</leftJoint>
 	    <rightJoint>right_wheel_joint</rightJoint>
 	    <wheelAcceleration>0</wheelAcceleration>
-	    <wheelTorque>1</wheelTorque>
+	    <wheelTorque>5</wheelTorque>
 	    <torque>1</torque>
 	    <commandTopic>cmd_vel</commandTopic>
@@ -183,4 +183,6 @@
 	    <rosDebugLevel>none</rosDebugLevel>
 	    <robotBaseFrame>base_link</robotBaseFrame>
+      <wheelSeparation>${wheel_separation}</wheelSeparation>
+      <wheelDiameter>${wheel_radius*2.0}</wheelDiameter>
 			<updateRate>10</updateRate>
 	  </plugin>
@@ -188,5 +190,5 @@
   <joint name="laser_joint" type="fixed">
     <axis xyz="0 1 0" />
-    <origin xyz="0 0 0.03" rpy="0 0 0"/>
+    <origin xyz="0 0 0.04" rpy="0 0 0"/>
     <parent link="body_link"/>
     <child link="laser_link"/>

Commit message: avoid laser scan hitting other kamagamis

File: urdf/kamagami.xacro (robot description, xacro)
@@ -129,8 +129,8 @@
 	<gazebo reference="raspicam_link">
 		<material>Gazebo/Grey</material>
-		<sensor type="camera" name="raspicam">
+		<sensor type="camera" name="camera">
 			<!--			<pose>0.089 -0.01 0.236 0 0.436 0</pose> -->
 			<update_rate>6.0</update_rate>
-			<camera name="raspicam">
+			<camera name="camera">
 				<horizontal_fov>1.0123</horizontal_fov>
 				<image>
@@ -152,5 +152,5 @@
 				<alwaysOn>true</alwaysOn>
 				<updateRate>0.0</updateRate>
-				<cameraName>raspicam</cameraName>
+				<cameraName>camera</cameraName>
 				<imageTopicName>image</imageTopicName>
 				<cameraInfoTopicName>camera_info</cameraInfoTopicName>
@@ -199,5 +199,5 @@
       <origin xyz="0 0 0" rpy="0 0 0"/>
       <geometry>
-    <box size="0.1 0.1 0.1"/>
+    <box size="0.001 0.001 0.001"/>
       </geometry>
     </collision>
@@ -210,5 +210,5 @@
     <gazebo reference="laser_link">
         <sensor name="laser" type="ray">
-        <pose>0 0 0 0 0 0</pose>
+        <pose>0 0 1 0 0 0</pose>
           <ray>
             <scan>
