Commit message: made cone transparent and red

File: urdf/kamagami_with_cone.xacro (robot description, xacro)
@@ -11,5 +11,16 @@
 </link>
 <gazebo reference="cone_link">
+  <visual name="cone_vis">
+  <transparency>0.8</transparency>
+  <material>
+  <ambient>1.0 0 0 0.1</ambient>
+  <diffuse>1.0 0 0 0.1</diffuse>
+  <specular>1.0 0 0 0.1</specular>
+  <emissive>1.0 0 0 0.1</emissive>
+  </material>
+  </visual>
+  <!--
 	<material value="Gazebo/YellowTransparent"/>
+  -->
 </gazebo>
 <joint name="cone_joint" type="fixed">
